File: _autosave-esp32-c3-02.kicad_sch (KiCad schematic)
At the start: 24 parts, among them J3 GSD090012SEU, J5 GSD090012SEU, U3 ESP32-C3-WROOM-02-H4, U4 CP2102N-A01-GQFN20R, U5 USBLC6-2SC6, U6 W25Q32JVSSIQ

Commit message: Connected USB to UART connector, ESP32 controller and the SD card module
Other:
- note added: "SD Card Module"
Changed lines of the file:
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@@
 	(generator_version "9.0")
 	(paper "A4")
+	(rectangle
+		(start 172.72 97.79)
+		(end 281.432 165.1)
+		(stroke
+			(width 0)
+			(type default)
+		)
+		(fill
+			(type none)
+		)
+	)
+	(text "SD Card Module"
+		(exclude_from_sim no)
+		(at 182.626 97.282 0)
+		(effects
+			(font
+				(size 1.27 1.27)
+			)
+		)
+	)
 	(text "ESP32 microcontroller"
 		(exclude_from_sim no)
