File: esp32-c3-02.kicad_sch (KiCad schematic)
At the start: 24 parts, among them J3 GSD090012SEU, J5 GSD090012SEU, U3 ESP32-C3-WROOM-02-H4, U4 CP2102N-A01-GQFN20R, U5 USBLC6-2SC6, U6 W25Q32JVSSIQ

Commit message: Finished schematic design; Still need to reassign the values to the capacitors and resistors
Parts:
- added C14: C, Capacitor_SMD:C_0805_2012Metric, symbol Device:C
- added R22: R, Resistor_SMD:R_0805_2012Metric, symbol Device:R
- added TP1, TP2, TP3, TP4, TP5: TestPoint, TestPoint:TestPoint_Pad_D1.0mm, symbol Connector:TestPoint
- C10, C13, C8: value 0.1u -> C; footprint (none) -> Capacitor_SMD:C_0805_2012Metric
- C11: value 1u -> C; footprint (none) -> Capacitor_SMD:C_0805_2012Metric
- C12, C7: value 10u -> C_Polarized
- C9: value 4.7u -> C_Polarized
- LED6: footprint (none) -> ESP32_IoT_Board_Footprint:LTST-C170GKT
- R11: value 1k -> R; footprint (none) -> Resistor_SMD:R_0805_2012Metric
- R12: value 22k1 -> R; footprint (none) -> Resistor_SMD:R_0805_2012Metric
- R13: value 47k5 -> R; footprint (none) -> Resistor_SMD:R_0805_2012Metric
- R14, R18: value 470 -> R; footprint (none) -> Resistor_SMD:R_0805_2012Metric
- R16, R20, R21: value 50 -> R; footprint (none) -> Resistor_SMD:R_0805_2012Metric
- R19: value 10k -> R; footprint (none) -> Resistor_SMD:R_0805_2012Metric
- U6: footprint (none) -> ESP32_IoT_Board_Footprint:W25Q32JVSSIQ
Connections:
- net +3.3V: now also U6.3 (~{WP}(IO2)), U6.7 (~{HOLD}/~{RESET}(IO3)), U6.8 (VCC), C14.1
- net CS: now also U6.1 (~{CS}), TP5.1
- net CS_SD: now also TP4.1
- net GND: now also U6.4 (GND), C14.2
- net MISO_DO: now also R22.1, TP2.1
- net MOSI_DI: now also U6.5 (DI(IO0)), TP1.1
- net SCLK: now also U6.6 (CLK), TP3.1
- net at U6.2 (DO(IO1)): now also R22.2
- net DTS renamed DTR
Other:
- added sheet Sensors (sensors.kicad_sch)
- added sheet User Interface (user_interface.kicad_sch)
- note added: "Flash Memory with SPI"
- note added: "SD Card Module with SPI interface"
- note added: "SPI interface test point"
- note removed: "SD Card Module"
- title: (none) -> ESP32 Controller and Memory Components
- moved on the sheet: C12, C13, U6
