File: iot_board.kicad_sch (KiCad schematic)
At the start: 25 parts, among them J1 SS-52400-003, J2 B2B-PH-SM4-TB, U2 MCP73871-2CAI_ML

Commit message: Finished schematic design; Still need to reassign the values to the capacitors and resistors
Parts:
- C1, C2, C5, C6: footprint (none) -> Capacitor_SMD:C_0805_2012Metric
- J1: Manufacturer Part Number (none) -> SS-52400-003
- LED2, LED4: footprint (none) -> ESP32_IoT_Board_Footprint:LTST-C170GKT
- R1, R2: value 10k -> R; footprint (none) -> Resistor_SMD:R_0805_2012Metric
- R10, R7, R8, R9: value 470 -> R; footprint (none) -> Resistor_SMD:R_0805_2012Metric
- R3, R4: value 5k1 -> R; footprint (none) -> Resistor_SMD:R_0805_2012Metric
- R5: value 2k -> R; footprint (none) -> Resistor_SMD:R_0805_2012Metric
- R6: value 20k -> R; footprint (none) -> Resistor_SMD:R_0805_2012Metric
Other:
- title: ESP32 sensor schematic -> ESP32 project schematic
Changed lines of the file:
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@@
 	(paper "A4")
 	(title_block
-		(title "ESP32 sensor schematic")
+		(title "ESP32 project schematic")
 		(date "2025-04-19")
 	)
@@
 			)
 		)
-		(property "Value" "2k"
+		(property "Value" "R"
 			(at 256.54 55.118 90)
 			(effects
@@
 			)
 		)
-		(property "Footprint" ""
+		(property "Footprint" "Resistor_SMD:R_0805_2012Metric"
 			(at 256.54 55.118 90)
 			(effects
@@
 			)
 		)
-		(property "Footprint" ""
+		(property "Footprint" "Capacitor_SMD:C_0805_2012Metric"
 			(at 108.9152 58.42 0)
 			(effects
@@
 			)
 		)
-		(property "Footprint" ""
+		(property "Footprint" "Capacitor_SMD:C_0805_2012Metric"
 			(at 180.0352 29.21 0)
 			(effects
@@
 			)
 		)
-		(property "Value" "470"
+		(property "Value" "R"
 			(at 170.18 58.4199 0)
 			(effects
@@
 			)
 		)
-		(property "Footprint" ""
+		(property "Footprint" "Resistor_SMD:R_0805_2012Metric"
 			(at 169.418 57.15 90)
 			(effects
@@
 			)
 		)
-		(property "Value" "10k"
+		(property "Value" "R"
 			(at 195.58 60.198 90)
 			(effects
@@
 			)
 		)
-		(property "Footprint" ""
+		(property "Footprint" "Resistor_SMD:R_0805_2012Metric"
 			(at 195.58 58.928 90)
 			(effects
@@
 			)
 		)
-		(property "Value" "20k"
+		(property "Value" "R"
 			(at 256.54 64.262 90)
 			(effects
@@
 			)
 		)
-		(property "Footprint" ""
+		(property "Footprint" "Resistor_SMD:R_0805_2012Metric"
 			(at 256.54 64.008 90)
 			(effects
@@
 			)
 		)
-		(property "Value" "10k"
+		(property "Value" "R"
 			(at 256.54 46.228 90)
 			(effects
@@
 			)
 		)
-		(property "Footprint" ""
+		(property "Footprint" "Resistor_SMD:R_0805_2012Metric"
 			(at 256.54 46.228 90)
 			(effects
@@
 			)
 		)
-		(property "Footprint" ""
+		(property "Footprint" "Capacitor_SMD:C_0805_2012Metric"
 			(at 39.0652 140.97 0)
 			(effects
@@
 			)
 		)
-		(property "Footprint" ""
+		(property "Footprint" "ESP32_IoT_Board_Footprint:LTST-C170GKT"
 			(at 196.85 147.955 0)
 			(effects
@@
 			)
 		)
-		(property "Value" "470"
+		(property "Value" "R"
 			(at 157.48 58.4199 0)
 			(effects
@@
 			)
 		)
-		(property "Footprint" ""
+		(property "Footprint" "Resistor_SMD:R_0805_2012Metric"
 			(at 156.718 57.15 90)
 			(effects
@@
 			)
 		)
-		(property "Footprint" ""
+		(property "Footprint" "Capacitor_SMD:C_0805_2012Metric"
 			(at 113.9952 139.7 0)
 			(effects
@@
 	)
 	(symbol
+		(lib_name "LTST-C170GKT_1")
 		(lib_id "ESP32_IoT_Board_Schem:LTST-C170GKT")
 		(at 180.34 64.77 90)
@@
 			)
 		)
-		(property "Footprint" ""
+		(property "Footprint" "ESP32_IoT_Board_Footprint:LTST-C170GKT"
 			(at 189.865 60.96 0)
 			(effects
@@
 			)
 		)
-		(property "Value" "5k1"
+		(property "Value" "R"
 			(at 25.4 58.4199 0)
 			(effects
@@
 			)
 		)
-		(property "Footprint" ""
+		(property "Footprint" "Resistor_SMD:R_0805_2012Metric"
 			(at 21.082 57.15 90)
 			(effects
@@
 			)
 		)
-		(property "Value" "470"
+		(property "Value" "R"
 			(at 182.88 58.4199 0)
 			(effects
@@
 			)
 		)
-		(property "Footprint" ""
+		(property "Footprint" "Resistor_SMD:R_0805_2012Metric"
 			(at 182.118 57.15 90)
 			(effects
@@
 			)
 		)
+		(property "Manufacturer Part Number" "SS-52400-003"
+			(at 66.04 88.9 0)
+			(effects
+				(font
+					(size 1.27 1.27)
+				)
+			)
+		)
 		(pin "A11"
 		)
@@
 			)
 		)
-		(property "Value" "470"
+		(property "Value" "R"
 			(at 199.3901 140.97 0)
 			(effects
@@
 			)
 		)
-		(property "Footprint" ""
+		(property "Footprint" "Resistor_SMD:R_0805_2012Metric"
 			(at 200.66 140.208 90)
 			(effects
@@
 			)
 		)
-		(property "Value" "5k1"
+		(property "Value" "R"
 			(at 100.33 59.6899 0)
 			(effects
@@
 			)
 		)
-		(property "Footprint" ""
+		(property "Footprint" "Resistor_SMD:R_0805_2012Metric"
 			(at 96.012 58.42 90)
 			(effects
